File: Mixer.kicad_pcb (KiCad board)
At the start: 2 copper layers, 99.1 x 57.2 mm, 39 parts, among them J1 Barrel_Jack, J2 AudioJack3, J3 AudioJack3, J4 AudioJack3, J5 AudioJack3, J6 AudioJack3, SW1 SW_SPST, U1 TL074

Commit message: Add gitignore and update PCB
Other:
- board text added: "PCB version 1.0"
- board text added: "STEREO AUDIO MIXER"
- board text added: "github.com/MaxTheWhale/stereo-mixer"
Changed lines of the file:
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@@
   (general
     (thickness 1.6)
-    (drawings 6)
+    (drawings 9)
     (tracks 174)
     (zones 0)
@@
   (page A4)
   (layers
-    (0 F.Cu signal)
-    (31 B.Cu signal)
+    (0 F.Cu signal hide)
+    (31 B.Cu signal hide)
     (32 B.Adhes user)
     (33 F.Adhes user)
@@
     (45 Margin user)
     (46 B.CrtYd user)
-    (47 F.CrtYd user)
+    (47 F.CrtYd user hide)
     (48 B.Fab user)
-    (49 F.Fab user)
+    (49 F.Fab user hide)
   )
   (setup
@@
     )
   )
+  (gr_text "STEREO AUDIO MIXER" (at 118.745 108.585) (layer F.SilkS)
+    (effects (font (size 2 2) (thickness 0.15)))
+  )
+  (gr_text "PCB version 1.0\n" (at 118.745 111.379) (layer F.SilkS)
+    (effects (font (size 1 1) (thickness 0.15)))
+  )
+  (gr_text github.com/MaxTheWhale/stereo-mixer (at 118.745 113.792) (layer F.SilkS)
+    (effects (font (size 1 1) (thickness 0.15)))
+  )
   (gr_line (start 166.37 83.82) (end 139.065 83.82) (layer Edge.Cuts) (width 0.05))

Commit message: Add libraries
Connections:
- R15 pad 1: Net-(C7-Pad2) -> Net-(R15-Pad1)
- RV5 pad 4: Net-(C7-Pad2) -> Net-(R15-Pad1)
- RV5 pad 5: Net-(C7-Pad2) -> Net-(R15-Pad1)
- U1 pad 8: Net-(U1-Pad8) -> Net-(C7-Pad2)
- U1 pad 9: Net-(C7-Pad2) -> Net-(R15-Pad1)
Routing:
- net Net-(C7-Pad2): track 38.4 -> 15.9 mm
- net Net-(R15-Pad1): track 0.00 -> 22.5 mm
- net Net-(J3-PadT): track 48.6 -> 50.9 mm
Changed lines of the file:
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@@
     (thickness 1.6)
     (drawings 9)
-    (tracks 174)
+    (tracks 176)
     (zones 0)
     (modules 39)
@@
   (page A4)
   (layers
-    (0 F.Cu signal hide)
-    (31 B.Cu signal hide)
+    (0 F.Cu signal)
+    (31 B.Cu signal)
     (32 B.Adhes user)
     (33 F.Adhes user)
@@
   (net 32 "Net-(J5-PadR)")
   (net 33 "Net-(J5-PadT)")
-  (net 34 "Net-(U1-Pad8)")
+  (net 34 "Net-(R15-Pad1)")
   (net_class Default "This is the default net class."
     (clearance 0.2)
@@
     (add_net "Net-(R13-Pad1)")
     (add_net "Net-(R14-Pad1)")
+    (add_net "Net-(R15-Pad1)")
     (add_net "Net-(R4-Pad2)")
     (add_net "Net-(R5-Pad2)")
@@
     (add_net "Net-(R8-Pad2)")
     (add_net "Net-(R9-Pad2)")
-    (add_net "Net-(U1-Pad8)")
     (add_net VREF)
   )
@@
     )
     (pad 4 thru_hole circle (at -5 0 270) (size 2.34 2.34) (drill 1.3) (layers *.Cu *.Mask)
-      (net 10 "Net-(C7-Pad2)"))
+      (net 34 "Net-(R15-Pad1)"))
     (pad 5 thru_hole circle (at -5 -5 270) (size 2.34 2.34) (drill 1.3) (layers *.Cu *.Mask)
-      (net 10 "Net-(C7-Pad2)"))
+      (net 34 "Net-(R15-Pad1)"))
     (pad 6 thru_hole circle (at -5 -10 270) (size 2.34 2.34) (drill 1.3) (layers *.Cu *.Mask)
       (net 10 "Net-(C7-Pad2)"))
@@
       (net 24 "Net-(R13-Pad1)"))
     (pad 1 thru_hole circle (at 0 0 180) (size 1.6 1.6) (drill 0.8) (layers *.Cu *.Mask)
-      (net 10 "Net-(C7-Pad2)"))
+      (net 34 "Net-(R15-Pad1)"))
     (model ${KISYS3DMOD}/Resistor_THT.3dshapes/R_Axial_DIN0207_L6.3mm_D2.5mm_P10.16mm_Horizontal.wrl
       (at (xyz 0 0 0))
@@
       (net 23 "Net-(R12-Pad1)"))
     (pad 8 thru_hole oval (at 7.62 15.24) (size 1.6 1.6) (drill 0.8) (layers *.Cu *.Mask)
-      (net 34 "Net-(U1-Pad8)"))
+      (net 10 "Net-(C7-Pad2)"))
     (pad 2 thru_hole oval (at 0 2.54) (size 1.6 1.6) (drill 0.8) (layers *.Cu *.Mask)
       (net 4 "Net-(C4-Pad1)"))
     (pad 9 thru_hole oval (at 7.62 12.7) (size 1.6 1.6) (drill 0.8) (layers *.Cu *.Mask)
-      (net 10 "Net-(C7-Pad2)"))
+      (net 34 "Net-(R15-Pad1)"))
     (pad 3 thru_hole oval (at 0 5.08) (size 1.6 1.6) (drill 0.8) (layers *.Cu *.Mask)
       (net 3 VREF))
@@
   (segment (start 155.02 123.11) (end 154.94 123.19) (width 0.25) (layer F.Cu) (net 10))
   (segment (start 161.29 123.11) (end 155.02 123.11) (width 0.25) (layer F.Cu) (net 10))
-  (segment (start 152.4 132.16) (end 157.4 132.16) (width 0.25) (layer F.Cu) (net 10))
-  (segment (start 154.94 120.65) (end 153.67 120.65) (width 0.25) (layer F.Cu) (net 10))
-  (segment (start 153.67 120.65) (end 152.4 121.92) (width 0.25) (layer F.Cu) (net 10))
-  (segment (start 152.4 121.92) (end 152.4 125.73) (width 0.25) (layer F.Cu) (net 10))
-  (segment (start 152.4 125.73) (end 153.67 127) (width 0.25) (layer F.Cu) (net 10))
-  (segment (start 156.464 127) (end 153.67 127) (width 0.25) (layer F.Cu) (net 10))
-  (segment (start 157.4 127.936) (end 157.4 128.698) (width 0.25) (layer F.Cu) (net 10))
-  (segment (start 156.464 127) (end 157.4 127.936) (width 0.25) (layer F.Cu) (net 10))
-  (segment (start 157.4 132.16) (end 157.4 128.698) (width 0.25) (layer F.Cu) (net 10))
-  (segment (start 157.4 128.698) (end 157.4 128.19) (width 0.25) (layer F.Cu) (net 10))
   (segment (start 161.29 118.11) (end 161.29 114.3) (width 0.25) (layer F.Cu) (net 11))
   (segment (start 161.29 114.3) (end 160.02 113.03) (width 0.25) (layer F.Cu) (net 11))
@@
   (segment (start 83.74 95.17) (end 81.2 92.63) (width 0.25) (layer B.Cu) (net 27))
   (segment (start 83.74 129.54) (end 83.74 95.17) (width 0.25) (layer B.Cu) (net 27))
-  (segment (start 97.79 129.54) (end 90.25 122) (width 0.25) (layer B.Cu) (net 28))
+  (segment (start 100.17 137.16) (end 97.757 134.747) (width 0.25) (layer B.Cu) (net 28))
   (segment (start 90.25 122) (end 90.25 92.63) (width 0.25) (layer B.Cu) (net 28))
-  (segment (start 100.17 137.16) (end 97.79 134.78) (width 0.25) (layer B.Cu) (net 28))
-  (segment (start 97.79 134.78) (end 97.79 129.54) (width 0.25) (layer B.Cu) (net 28))
+  (segment (start 97.757 134.747) (end 93.853 134.747) (width 0.25) (layer B.Cu) (net 28))
+  (segment (start 92.71 133.604) (end 92.71 124.46) (width 0.25) (layer B.Cu) (net 28))
+  (segment (start 93.853 134.747) (end 92.71 133.604) (width 0.25) (layer B.Cu) (net 28))
+  (segment (start 92.71 124.46) (end 90.25 122) (width 0.25) (layer B.Cu) (net 28))
   (segment (start 100.25 132.08) (end 100.25 92.63) (width 0.25) (layer B.Cu) (net 29))
   (segment (start 100.17 132.16) (end 100.25 132.08) (width 0.25) (layer B.Cu) (net 29))
@@
   (segment (start 135.73 134.62) (end 131.826 134.62) (width 0.25) (layer B.Cu) (net 33))
   (segment (start 131.826 134.62) (end 130.81 133.604) (width 0.25) (layer B.Cu) (net 33))
+  (segment (start 152.4 132.16) (end 157.4 132.16) (width 0.25) (layer F.Cu) (net 34))
+  (segment (start 154.94 120.65) (end 153.67 120.65) (width 0.25) (layer F.Cu) (net 34))
+  (segment (start 153.67 120.65) (end 152.4 121.92) (width 0.25) (layer F.Cu) (net 34))
+  (segment (start 152.4 121.92) (end 152.4 125.73) (width 0.25) (layer F.Cu) (net 34))
+  (segment (start 152.4 125.73) (end 153.67 127) (width 0.25) (layer F.Cu) (net 34))
+  (segment (start 156.464 127) (end 153.67 127) (width 0.25) (layer F.Cu) (net 34))
+  (segment (start 157.4 127.936) (end 157.4 128.698) (width 0.25) (layer F.Cu) (net 34))
+  (segment (start 156.464 127) (end 157.4 127.936) (width 0.25) (layer F.Cu) (net 34))
+  (segment (start 157.4 132.16) (end 157.4 128.698) (width 0.25) (layer F.Cu) (net 34))
+  (segment (start 157.4 128.698) (end 157.4 128.19) (width 0.25) (layer F.Cu) (net 34))
   (zone (net 1) (net_name Earth) (layer B.Cu) (hatch edge 0.508)
     (connect_pads (clearance 0.508))

Commit message: Update PCB to v1.1
Parts:
- added C1: 220u, Capacitor_THT:CP_Radial_D6.3mm_P2.50mm, F.Cu at (87.0, 101.6)
- moved C3 26.7 mm to (114.3, 97.8)
- moved C7 5.08 mm to (156.2, 102.9), turned to 90 degrees
- moved C8 5.08 mm to (161.3, 123.2), turned to 90 degrees
- renumbered C1 to C2, C2 to C3, C3 to C4, C4 to C5, C5 to C6, C6 to C7, C7 to C8
Connections:
- C7 pad 1: Net-(C6-Pad1) (its old number) -> Net-(C7-Pad1)
- C7 pad 2: Net-(C6-Pad2) (its old number) -> Net-(C7-Pad2)
- C8 pad 1: Net-(C7-Pad1) -> Net-(C8-Pad1)
- C8 pad 2: Net-(C7-Pad2) -> Net-(C8-Pad2)
- J6 pad R: Net-(C7-Pad1) -> Net-(C8-Pad2)
- J6 pad T: Net-(C6-Pad1) (its old number) -> Net-(C7-Pad2)
- R16 pad 2: Net-(C6-Pad1) (its old number) -> Net-(C7-Pad2)
- R17 pad 2: Net-(C7-Pad1) -> Net-(C8-Pad2)
- RV5 pad 1: Net-(R14-Pad1) -> Net-(C7-Pad1)
- RV5 pad 3: Net-(C6-Pad2) (its old number) -> Net-(R14-Pad1)
- RV5 pad 4: Net-(R15-Pad1) -> Net-(C8-Pad1)
- RV5 pad 6: Net-(C7-Pad2) -> Net-(R15-Pad1)
- U1 pad 14: Net-(C6-Pad2) (its old number) -> Net-(C7-Pad1)
- U1 pad 8: Net-(C7-Pad2) -> Net-(C8-Pad1)
Routing:
- net Net-(C6-Pad2) (its old number): track 38.0 -> 0.00 mm
- net Net-(C8-Pad2): track 0.00 -> 27.1 mm
- net Net-(C8-Pad1): track 0.00 -> 16.5 mm
- net Net-(C1-Pad1): track 9.73 -> 26.1 mm
- net Net-(C6-Pad1) (its old number): track 13.6 -> 0.00 mm
- net Net-(C7-Pad1): track 27.1 -> 38.1 mm
- net VREF: track 92.3 -> 84.4 mm
- net Net-(R14-Pad1): track 42.8 -> 47.0 mm
- net Net-(C7-Pad2): track 15.9 -> 13.6 mm
- net Net-(R15-Pad1): track 22.5 -> 22.0 mm
Other:
- board text added: "9V DC"
- board text added: "PCB version 1.1"
- board text removed: "PCB version 1.0"
