File: Mixer.sch (KiCad schematic (older format))
At the start: 39 parts, among them J1 Barrel_Jack, J2 AudioJack3, J3 AudioJack3, J4 AudioJack3, J5 AudioJack3, J6 AudioJack3, SW1 SW_SPST, U1 TL074

Commit message: Add libraries
Changed lines of the file:
@@
 	2200 1650 1050 1650
-Wire Wire Line
-	1050 1550 1200 1550
-Wire Wire Line
-	1200 1550 1200 2050
 Wire Wire Line
 	1200 2050 1400 2050
@@
 Wire Wire Line
 	2300 3450 2400 3450
-Wire Wire Line
-	1200 1350 1200 1550
 Connection ~ 1200 1350
-Connection ~ 1200 1550
 Wire Wire Line
 	1200 2050 1200 2250
@@
 	5300 2850 5500 2850
 Wire Wire Line
-	3600 3400 -1100 3400
-Wire Wire Line
-	-1100 3400 -1100 8700
-Wire Wire Line
 	6100 2750 6450 2750
 Connection ~ 6450 2750
 Wire Wire Line
 	6450 2750 6450 3250
+Wire Wire Line
+	1200 1350 1200 1550
+Wire Wire Line
+	1050 1550 1200 1550
+Connection ~ 1200 1550
+Wire Wire Line
+	1200 1550 1200 2050
+Text Label 1550 5150 0    50   ~ 0
+GND
 $EndSCHEMATC

Commit message: Update PCB to v1.1
Parts:
- added C1: 220u, Capacitor_THT:CP_Radial_D6.3mm_P2.50mm, symbol Device:CP
- renumbered C1 to C2, C2 to C3, C3 to C4, C4 to C5, C5 to C6, C6 to C7, C7 to C8
Connections:
- net Earth: now also C1.2
- net at R14.1, RV5.2, U1.13 (-): now also RV5.3; no longer RV5.1
- net at R15.1, RV5.5, U1.9 (-): now also RV5.6; no longer RV5.4
- net at J6.T, R16.2: now also C7.2; no longer C7.1
- net at J6.R, R17.2: now also C8.2; no longer C8.1
- net at D1.2 (A), SW1.2 (B): now also C1.1
- new net: C7.1, RV5.1, U1.14
- new net: C8.1, RV5.4, U1.8
Other:
- moved on the sheet: C2
Changed lines of the file:
@@
 	4800 1650 4950 1650
 $Comp
-L Device:CP C4
+L Device:CP C5
 U 1 1 5F4B5672
 P 3600 1750
-F 0 "C4" V 3345 1750 50  0000 C CNN
+F 0 "C5" V 3345 1750 50  0000 C CNN
 F 1 "10u" V 3436 1750 50  0000 C CNN
 F 2 "Capacitor_THT:CP_Radial_Tantal_D4.5mm_P5.00mm" H 3638 1600 50  0001 C CNN
@@
 Connection ~ 3950 1750
 $Comp
-L Device:CP C5
+L Device:CP C6
 U 1 1 5F4BCA07
 P 3600 2950
-F 0 "C5" V 3345 2950 50  0000 C CNN
+F 0 "C6" V 3345 2950 50  0000 C CNN
 F 1 "10u" V 3436 2950 50  0000 C CNN
 F 2 "Capacitor_THT:CP_Radial_Tantal_D4.5mm_P5.00mm" H 3638 2800 50  0001 C CNN
@@
 Wire Wire Line
 	4000 1550 4000 1300
-$Comp
-L Device:R_POT_Dual RV5
-U 1 1 5F4C70AA
-P 6550 2150
-F 0 "RV5" V 6504 1963 50  0000 R CNN
-F 1 "100k" V 6595 1963 50  0000 R CNN
-F 2 "Potentiometer_THT:Potentiometer_Alps_RK163_Dual_Horizontal" H 6800 2075 50  0001 C CNN
-F 3 "~" H 6800 2075 50  0001 C CNN
-	1    6550 2150
-	0    1    1    0
-$EndComp
 Connection ~ 5400 1650
 Wire Wire Line
@@
 Wire Wire Line
 	3300 1750 3450 1750
-Wire Wire Line
-	6650 1900 6650 1750
-Wire Wire Line
-	6650 1750 6450 1750
-Wire Wire Line
-	6650 2400 6650 2250
-Wire Wire Line
-	6650 2250 6450 2250
-Wire Wire Line
-	6450 1750 5400 1750
-Connection ~ 6450 1750
-Wire Wire Line
-	5400 1750 5400 1650
-Wire Wire Line
-	6450 2250 5300 2250
-Wire Wire Line
-	5300 2250 5300 2850
-Connection ~ 6450 2250
 Connection ~ 5300 2850
-Wire Wire Line
-	6450 2050 6750 2050
-Wire Wire Line
-	6750 2050 6750 1550
-Wire Wire Line
-	6100 1550 6750 1550
-Wire Wire Line
-	6450 2550 6450 2750
-$Comp
-L Device:CP C6
+$Comp
+L Device:CP C7
 U 1 1 5F4B8CC6
 P 7050 1550
-F 0 "C6" V 6795 1550 50  0000 C CNN
+F 0 "C7" V 6795 1550 50  0000 C CNN
 F 1 "10u" V 6886 1550 50  0000 C CNN
 F 2 "Capacitor_THT:CP_Radial_Tantal_D4.5mm_P5.00mm" H 7088 1400 50  0001 C CNN
 F 3 "~" H 7050 1550 50  0001 C CNN
 	1    7050 1550
-	0    1    1    0
-$EndComp
-$Comp
-L Device:CP C7
-U 1 1 5F4B9B94
-P 7050 3250
-F 0 "C7" V 6795 3250 50  0000 C CNN
-F 1 "10u" V 6886 3250 50  0000 C CNN
-F 2 "Capacitor_THT:CP_Radial_Tantal_D4.5mm_P5.00mm" H 7088 3100 50  0001 C CNN
-F 3 "~" H 7050 3250 50  0001 C CNN
-	1    7050 3250
-	0    1    1    0
-$EndComp
-Wire Wire Line
-	6750 1550 6900 1550
-Connection ~ 6750 1550
+	0    -1   -1   0
+$EndComp
 Wire Wire Line
 	6450 3250 6900 3250
@@
 Wire Wire Line
 	1950 4200 1900 4200
-Connection ~ 2250 4200
 $Comp
 L Switch:SW_SPST SW1
@@
 Connection ~ 3600 4200
 $Comp
-L Device:C C3
+L Device:C C4
 U 1 1 5F512172
 P 4000 4550
-F 0 "C3" H 4115 4596 50  0000 L CNN
+F 0 "C4" H 4115 4596 50  0000 L CNN
 F 1 "100n" H 4115 4505 50  0000 L CNN
 F 2 "Capacitor_THT:C_Disc_D7.0mm_W2.5mm_P5.00mm" H 4038 4400 50  0001 C CNN
@@
 $EndComp
 Wire Wire Line
-	2250 4900 2800 4900
-Connection ~ 2250 4900
-Wire Wire Line
-	2250 4700 2250 4900
-Wire Wire Line
-	1550 4900 2250 4900
-Wire Wire Line
-	2250 4200 3100 4200
-Wire Wire Line
-	2250 4200 2250 4400
+	2350 4700 2350 4900
+Wire Wire Line
+	2250 4200 2350 4200
+Wire Wire Line
+	2350 4200 2350 4400
 Connection ~ 2800 4900
 Wire Wire Line
@@
 Wire Wire Line
 	3100 4600 3100 4550
-Wire Wire Line
-	1550 4400 1550 4900
 Wire Wire Line
 	1550 4900 1550 5150
@@
 $EndComp
 $Comp
-L Device:CP C2
+L Device:CP C3
 U 1 1 5F4E9910
 P 2800 4700
-F 0 "C2" V 2545 4700 50  0000 C CNN
+F 0 "C3" V 2545 4700 50  0000 C CNN
 F 1 "10u" V 2636 4700 50  0000 C CNN
 F 2 "Capacitor_THT:CP_Radial_Tantal_D4.5mm_P5.00mm" H 2838 4550 50  0001 C CNN
@@
 $EndComp
 $Comp
-L Device:CP C1
+L Device:CP C2
 U 1 1 5F4DC898
-P 2250 4550
-F 0 "C1" V 1995 4550 50  0000 C CNN
-F 1 "10u" V 2086 4550 50  0000 C CNN
-F 2 "Capacitor_THT:CP_Radial_Tantal_D4.5mm_P5.00mm" H 2288 4400 50  0001 C CNN
-F 3 "~" H 2250 4550 50  0001 C CNN
-	1    2250 4550
+P 2350 4550
+F 0 "C2" V 2095 4550 50  0000 C CNN
+F 1 "10u" V 2186 4550 50  0000 C CNN
+F 2 "Capacitor_THT:CP_Radial_Tantal_D4.5mm_P5.00mm" H 2388 4400 50  0001 C CNN
+F 3 "~" H 2350 4550 50  0001 C CNN
+	1    2350 4550
 	1    0    0    -1
 $EndComp
@@
 	5300 2850 5500 2850
 Wire Wire Line
-	6100 2750 6450 2750
-Connection ~ 6450 2750
+	6100 2750 6300 2750
 Wire Wire Line
 	6450 2750 6450 3250
@@
 Text Label 1550 5150 0    50   ~ 0
 GND
+$Comp
+L Device:CP C1
+U 1 1 5F685EF5
+P 1900 4750
+F 0 "C1" H 2018 4796 50  0000 L CNN
+F 1 "220u" H 2018 4705 50  0000 L CNN
+F 2 "Capacitor_THT:CP_Radial_D6.3mm_P2.50mm" H 1938 4600 50  0001 C CNN
+F 3 "~" H 1900 4750 50  0001 C CNN
+	1    1900 4750
+	1    0    0    -1
+$EndComp
+Wire Wire Line
+	1550 4400 1550 4900
+Connection ~ 1900 4200
+Connection ~ 2350 4200
+Wire Wire Line
+	2350 4200 3100 4200
+Connection ~ 2350 4900
+Wire Wire Line
+	2350 4900 2800 4900
+Connection ~ 1900 4900
+Wire Wire Line
+	1900 4900 2350 4900
+Wire Wire Line
+	1550 4900 1900 4900
+Wire Wire Line
+	1900 4200 1900 4600
+$Comp
+L Device:CP C8
+U 1 1 5F4B9B94
+P 7050 3250
+F 0 "C8" V 6795 3250 50  0000 C CNN
+F 1 "10u" V 6886 3250 50  0000 C CNN
+F 2 "Capacitor_THT:CP_Radial_Tantal_D4.5mm_P5.00mm" H 7088 3100 50  0001 C CNN
+F 3 "~" H 7050 3250 50  0001 C CNN
+	1    7050 3250
+	0    -1   -1   0
+$EndComp
+Wire Wire Line
+	6450 2550 6650 2550
+Wire Wire Line
+	6650 2200 5300 2200
+Wire Wire Line
+	5300 2200 5300 2850
+Wire Wire Line
+	6450 2250 6300 2250
+Wire Wire Line
+	6300 2250 6300 2750
+Connection ~ 6300 2750
+Wire Wire Line
+	6300 2750 6450 2750
+Wire Wire Line
+	6650 2200 6650 2400
+Wire Wire Line
+	6650 2550 6650 2400
+Connection ~ 6650 2400
+$Comp
+L Device:R_POT_Dual RV5
+U 1 1 5F4C70AA
+P 6550 2150
+F 0 "RV5" V 6504 1963 50  0000 R CNN
+F 1 "100k" V 6595 1963 50  0000 R CNN
+F 2 "Potentiometer_THT:Potentiometer_Alps_RK163_Dual_Horizontal" H 6800 2075 50  0001 C CNN
+F 3 "~" H 6800 2075 50  0001 C CNN
+	1    6550 2150
+	0    1    1    0
+$EndComp
+Wire Wire Line
+	6100 1550 6450 1550
+Wire Wire Line
+	6450 1750 6450 1550
+Connection ~ 6450 1550
+Wire Wire Line
+	6450 1550 6900 1550
+Wire Wire Line
+	6650 1900 6650 2050
+Wire Wire Line
+	6650 2050 6450 2050
+Wire Wire Line
+	5400 2050 6450 2050
+Wire Wire Line
+	5400 1650 5400 2050
+Connection ~ 6450 2050
 $EndSCHEMATC
